File: led-array.kicad_pcb (KiCad board)
At the start: 4 copper layers, 180 x 105 mm, 1226 parts, among them J1 Conn_01x04_Pin, J2 USB_B_Micro, Q1 Q_NMOS_GDS, Q2 Q_NMOS_GDS, Q3 Q_NMOS_GDS, Q4 Q_NMOS_GDS, Q5 Q_NMOS_GDS, Q6 Q_NMOS_GDS, Q7 Q_NMOS_GDS, Q8 Q_NMOS_GDS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

Commit message: Actually hopefully final
Routing:
- net GND: track 68.3 -> 58.7 mm
- net K7: vias 7 -> 3
- net K6: vias 6 -> 2
- net K5: vias 6 -> 2
- net K4: vias 6 -> 2
- net K3: vias 6 -> 2
- net K2: vias 6 -> 2
- net /LED Group 3/Led Module 3/A3: vias 9 -> 1
- net /LED Group 3/Led Module 3/A2: vias 9 -> 1
- net /LED Group 3/Led Module 3/A1: vias 9 -> 1
- net /LED Group 3/Led Module 3/A0: vias 9 -> 1
- net /LED Group 3/Led Module 2/A7: vias 9 -> 1
- net /LED Group 3/Led Module 2/A6: vias 9 -> 1
- net /LED Group 3/Led Module 2/A5: vias 9 -> 1
- net /LED Group 3/Led Module 2/A4: vias 9 -> 1
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