File: led-array.kicad_pcb (KiCad board)
At the start: 4 copper layers, 180 x 105 mm, 1226 parts, among them J1 Conn_01x04_Pin, J2 USB_B_Micro, Q1 Q_NMOS_GDS, Q2 Q_NMOS_GDS, Q3 Q_NMOS_GDS, Q4 Q_NMOS_GDS, Q5 Q_NMOS_GDS, Q6 Q_NMOS_GDS, Q7 Q_NMOS_GDS, Q8 Q_NMOS_GDS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

Commit message: PCB laid out
Parts:
- moved R2 1.41 mm to (117.1, 172.6)
- moved R3 0.92 mm to (111.8, 172.6)
- moved C5 0.80 mm to (123.2, 165.7)
Connections:
- C3 pad 1: Net-(U1-PH) -> +3.3V
Routing:
- net +3.3V: track 653.4 -> 669.3 mm
- net Net-(U1-PH): track 5.85 -> 3.38 mm
- net K2: track 495.8 -> 495.6 mm, vias 2 -> 6
- net K6: vias 2 -> 6
- net K3: vias 2 -> 6
- net K7: vias 3 -> 7
- net K5: vias 2 -> 6
- net K4: vias 2 -> 6
- net /LED Group 3/Led Module 3/A3: vias 1 -> 9
- net /LED Group 3/Led Module 3/A2: vias 1 -> 9
- net /LED Group 3/Led Module 3/A1: vias 1 -> 9
- net /LED Group 3/Led Module 3/A0: vias 1 -> 9
- net /LED Group 3/Led Module 2/A7: vias 1 -> 9
- net /LED Group 3/Led Module 2/A6: vias 1 -> 9
- net /LED Group 3/Led Module 2/A5: vias 1 -> 9
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