File: _autosave-led-array.kicad_sch (KiCad schematic)
At the start: 42 parts, among them J1 Conn_01x04_Pin, J2 USB_B_Micro, Q1 Q_NMOS_GDS, Q2 Q_NMOS_GDS, Q3 Q_NMOS_GDS, Q4 Q_NMOS_GDS, Q5 Q_NMOS_GDS, Q6 Q_NMOS_GDS, Q7 Q_NMOS_GDS, Q8 Q_NMOS_GDS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

Commit message: PCB laid out
Other:
- note added: "MOUNTING HOLES"
- moved on the sheet: H1, H2, H3, H4
Changed lines of the file:
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@@
 	)
 	(rectangle
-		(start 60.96 226.06)
-		(end 134.62 261.62)
+		(start 147.32 190.5)
+		(end 205.74 213.36)
 		(stroke
 			(width 0)
@@
 		)
 	)
+	(text "MOUNTING HOLES"
+		(exclude_from_sim no)
+		(at 164.338 187.706 0)
+		(effects
+			(font
+				(size 2.54 2.54)
+			)
+		)
+	)
 	(text "LED GROUPS"
 		(exclude_from_sim no)
@@
 	(symbol
 		(lib_id "Mechanical:MountingHole")
-		(at 67.31 231.14 0)
+		(at 153.67 195.58 0)
 		(unit 1)
 		(exclude_from_sim no)
@@
 		(fields_autoplaced yes)
 		(property "Reference" "H4"
-			(at 69.85 229.8699 0)
+			(at 156.21 194.3099 0)
 			(effects
 				(font
@@
 		)
 		(property "Value" "MountingHole"
-			(at 69.85 232.4099 0)
+			(at 156.21 196.8499 0)
 			(effects
 				(font
@@
 		)
 		(property "Footprint" "MountingHole:MountingHole_3.2mm_M3"
-			(at 67.31 231.14 0)
+			(at 153.67 195.58 0)
 			(effects
 				(font
@@
 		)
 		(property "Datasheet" "~"
-			(at 67.31 231.14 0)
+			(at 153.67 195.58 0)
 			(effects
 				(font
@@
 		)
 		(property "Description" "Mounting Hole without connection"
-			(at 67.31 231.14 0)
+			(at 153.67 195.58 0)
 			(effects
 				(font
@@
 	(symbol
 		(lib_id "Mechanical:MountingHole")
-		(at 67.31 243.84 0)
+		(at 153.67 208.28 0)
 		(unit 1)
 		(exclude_from_sim no)
@@
 		(fields_autoplaced yes)
 		(property "Reference" "H1"
-			(at 69.85 242.5699 0)
+			(at 156.21 207.0099 0)
 			(effects
 				(font
@@
 		)
 		(property "Value" "MountingHole"
-			(at 69.85 245.1099 0)
+			(at 156.21 209.5499 0)
 			(effects
 				(font
@@
 		)
 		(property "Footprint" "MountingHole:MountingHole_3.2mm_M3"
-			(at 67.31 243.84 0)
+			(at 153.67 208.28 0)
 			(effects
 				(font
@@
 		)
 		(property "Datasheet" "~"
-			(at 67.31 243.84 0)
+			(at 153.67 208.28 0)
 			(effects
 				(font
@@
 		)
 		(property "Description" "Mounting Hole without connection"
-			(at 67.31 243.84 0)
+			(at 153.67 208.28 0)
 			(effects
 				(font
@@
 	(symbol
 		(lib_id "Mechanical:MountingHole")
-		(at 91.44 243.84 0)
+		(at 177.8 208.28 0)
 		(unit 1)
 		(exclude_from_sim no)
@@
 		(fields_autoplaced yes)
 		(property "Reference" "H3"
-			(at 93.98 242.5699 0)
+			(at 180.34 207.0099 0)
 			(effects
 				(font
@@
 		)
 		(property "Value" "MountingHole"
-			(at 93.98 245.1099 0)
+			(at 180.34 209.5499 0)
 			(effects
 				(font
@@
 		)
 		(property "Footprint" "MountingHole:MountingHole_3.2mm_M3"
-			(at 91.44 243.84 0)
+			(at 177.8 208.28 0)
 			(effects
 				(font
@@
 		)
 		(property "Datasheet" "~"
-			(at 91.44 243.84 0)
+			(at 177.8 208.28 0)
 			(effects
 				(font
@@
 		)
 		(property "Description" "Mounting Hole without connection"
-			(at 91.44 243.84 0)
+			(at 177.8 208.28 0)
 			(effects
 				(font
@@
 	(symbol
 		(lib_id "Mechanical:MountingHole")
-		(at 91.44 231.14 0)
+		(at 177.8 195.58 0)
 		(unit 1)
 		(exclude_from_sim no)
@@
 		(fields_autoplaced yes)
 		(property "Reference" "H2"
-			(at 93.98 229.8699 0)
+			(at 180.34 194.3099 0)
 			(effects
 				(font
@@
 		)
 		(property "Value" "MountingHole"
-			(at 93.98 232.4099 0)
+			(at 180.34 196.8499 0)
 			(effects
 				(font
@@
 		)
 		(property "Footprint" "MountingHole:MountingHole_3.2mm_M3"
-			(at 91.44 231.14 0)
+			(at 177.8 195.58 0)
 			(effects
 				(font
@@
 		)
 		(property "Datasheet" "~"
-			(at 91.44 231.14 0)
+			(at 177.8 195.58 0)
 			(effects
 				(font
@@
 		)
 		(property "Description" "Mounting Hole without connection"
-			(at 91.44 231.14 0)
+			(at 177.8 195.58 0)
 			(effects
 				(font
