File: _autosave-led-array.kicad_pcb (KiCad board)
At the start: 4 copper layers, 180 x 105 mm, 1227 parts, among them J1 Conn_01x04_Pin, J2 USB_B_Micro, Q1 Q_NMOS_GDS, Q2 Q_NMOS_GDS, Q3 Q_NMOS_GDS, Q4 Q_NMOS_GDS, Q5 Q_NMOS_GDS, Q6 Q_NMOS_GDS, Q7 Q_NMOS_GDS, Q8 Q_NMOS_GDS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

Commit message: Updated schematic, still likely need to modify the buck converter
Parts:
- C5: value 25u -> 22u
Changed lines of the file:
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@@
 			(usegerberattributes yes)
 			(usegerberadvancedattributes yes)
-			(creategerberjobfile yes)
+			(creategerberjobfile no)
 			(dashed_line_dash_ratio 12.000000)
 			(dashed_line_gap_ratio 3.000000)
@@
 			(drillshape 0)
 			(scaleselection 1)
-			(outputdirectory "Gerbers/")
+			(outputdirectory "Assembly/")
 		)
 	)
@@
 			)
 		)
-		(property "Value" "25u"
+		(property "Value" "22u"
 			(at 0 1.68 0)
 			(layer "F.Fab")
